File: THE DIMMER _ M4SDRV.kicad_sch (KiCad schematic)
At the start: 81 parts, among them J1 Conn_01x01, J10 GS2, J2 USB_B_Micro, J3 Conn_01x05, J4 Conn_01x02, J5 Conn_01x01, J6 Conn_01x01, J7 Conn_01x04, J8 Conn_01x02, J9 Conn_01x04, U1 ATSAMD51J19A-M, U10 DRV50153A, U11 DRV50152A, U12 Si8540, U13 Si8540, U14 TMC2209-LA, U3 ST730M50R, U4 BSC0925NDATMA1, U5 BSC0925NDATMA1, U6 BSC0925NDATMA1, U7 Si8540, U8 NCP170, U9 DRV50152A, Y1 Crystal_GND2_Small

Commit message: Added curretn sensor and driver
Added current sensor MAX40056 and MOSFET driver MIC4605-2YMT.
Parts:
- removed R10, R14, R18: 2k, Resistor_SMD:R_0603_1608Metric_Pad1.05x0.95mm_HandSolder, symbol device:R_Small
- removed R11, R13, R15, R17, R7, R9: 100ohm, Resistor_SMD:R_0603_1608Metric_Pad1.05x0.95mm_HandSolder, symbol device:R_Small
- removed R12, R16: 0.02ohm, Resistor_SMD:R_0805_2012Metric_Pad1.15x1.40mm_HandSolder, symbol device:R_Small
- removed U12, U13, U7: Si8540, Package_TO_SOT_SMD:SOT-23-5_HandSoldering, symbol si8540:Si8540
- removed U3: ST730M50R, Package_TO_SOT_SMD:SOT-23-5, symbol st730m50r:ST730M50R
- added C32, C33, C34, C35, C36, C37: 1uF, Capacitor_SMD:C_0603_1608Metric, symbol device:C
- added C38, C40, C42: 10nF, Capacitor_SMD:C_0402_1005Metric, symbol device:C
- added C39, C41, C43: 1uF, Capacitor_SMD:C_0402_1005Metric, symbol device:C
- added R2, R3: 0.02ohm, Resistor_SMD:R_0805_2012Metric_Pad1.15x1.40mm_HandSolder, symbol device:R_Small
- added U12, U13, U7: MAX40056_uMAX8, symbol max40056_umax8:MAX40056_uMAX8
- added U15, U16, U2: MIC4605-2YMT, Package_DFN_QFN:TDFN-10-1EP_2x3mm_P0.5mm_EP0.9x2mm, symbol mic4605-2ymtv2:MIC4605-2YMT
- added U3: LM2672M-12, Package_SO:SOIC-8_3.9x4.9mm_P1.27mm, symbol dc-dc:LM2672M-12
Connections:
- net +12V: now also J10.1 (G1), C32.1, C33.1, C34.1, R2.1, R2.2, R3.1, R3.2, U12.1 (¨RS+), U12.8 (RS), U13.1 (¨RS+), U13.8 (RS), U15.2 (VDD), U16.2 (VDD), U2.2 (VDD), U3.1 (CB), U7.1 (¨RS+), U7.8 (RS)
- net +3V3: now also C38.2, C39.2, C40.2, C41.2, C42.2, C43.2, U12.3 (VDD), U13.3 (VDD), U15.1 (EN), U16.1 (EN), U2.1 (EN), U7.3 (VDD)
- net A2: now also U12.4 (OUT)
- net A3: now also U13.4 (OUT)
- net A6: now also U7.4 (OUT)
- net GND: now also C32.2, C33.2, C34.2, C38.1, C39.1, C40.1, C41.1, C42.1, C43.1, U12.6 (GND), U13.6 (GND), U15.8 (VSS), U16.8 (VSS), U2.8 (VSS), U3.6 (GND), U7.6 (GND)
- net TCC0_CH0/Switch 1: now also U2.6 (PWM); no longer U4.8 (G2(GLD))
- net TCC0_CH1/Switch 2: no longer U4.1 (G1(GHS))
- net TCC0_CH2/Switch 3: no longer U5.8 (G2(GLD))
- net TCC0_CH3/Switch 4: now also U15.6 (PWM); no longer U5.1 (G1(GHS))
- net TCC0_CH4/Switch 5: no longer U6.8 (G2(GLD))
- net TCC0_CH5/Switch 6: now also U16.6 (PWM); no longer U6.1 (G1(GHS))
- net U: now also C37.2, U16.5 (HS)
- net V: now also C36.2, U15.5 (HS)
- net W: now also C35.2, U2.5 (HS)
- new net: C36.1, U15.3 (HB)
- new net: C35.1, U2.3 (HB)
- new net: C37.1, U16.3 (HB)
- new net HB1_HO: U2.4 (HO), U4.1 (G1(GHS))
- new net HB1_LO: U2.9 (LO), U4.8 (G2(GLD))
- new net HB2_HO: U15.4 (HO), U5.1 (G1(GHS))
- new net HB2_LO: U15.9 (LO), U5.8 (G2(GLD))
- new net HB3_HO: U16.4 (HO), U6.1 (G1(GHS))
- new net HB3_LO: U16.9 (LO), U6.8 (G2(GLD))
- new net VIN MAX 24V: U3.7 (VIN)
Other:
- moved on the sheet: R8

Commit message: update
Parts:
- added C44, C45: 1uF, Capacitor_SMD:C_0603_1608Metric, symbol device:C
- added J11: Conn_01x01, Connector_PinHeader_2.54mm:PinHeader_1x01_P2.54mm_Vertical, symbol conn:Conn_01x01
- added J12: Conn_01x02, Connector_PinHeader_1.27mm:PinHeader_1x02_P1.27mm_Vertical, symbol conn:Conn_01x02
- added U17: MIC4605-2YMT, Package_DFN_QFN:TDFN-10-1EP_2x3mm_P0.5mm_EP0.9x2mm, symbol mic4605-2ymtv2:MIC4605-2YMT
- added U18: BSC0925NDATMA1, Package_SON:Infineon_PG-TISON-8-2, symbol bsc0925ndatma1:BSC0925NDATMA1
Connections:
- net +12V: now also C44.1, U17.2 (VDD), U18.2 (D1(Vin)), U18.3 (D1(Vin)), U18.4 (D1(Vin)); no longer R2.1, R2.2, R3.1, R3.2, R8.1, R8.2, U12.1 (¨RS+), U12.8 (RS), U13.1 (¨RS+), U13.8 (RS), U7.1 (¨RS+), U7.8 (RS)
- net +3V3: now also U17.1 (EN)
- net A2: now also U7.4 (OUT); no longer U12.4 (OUT)
- net A6: now also U12.4 (OUT); no longer U7.4 (OUT)
- net CAN1_RX: now also U1.28 (PB15); no longer U1.26 (PB13)
- net CAN1_TX: now also U1.27 (PB14); no longer U1.25 (PB12)
- net GND: now also C44.2, U17.8 (VSS), U18.5 (S2(gnd)), U18.6 (S2(gnd)), U18.7 (S2(gnd))
- net TCC0_CH1/Switch 2: now also U17.6 (PWM)
- net U: now also R3.1, R3.2, U13.1 (¨RS+), U13.8 (RS)
- net UART_RX: now also J12.2 (Pin_2)
- net UART_TX: now also J12.1 (Pin_1)
- net V: now also R2.1, R2.2, U12.1 (¨RS+), U12.8 (RS)
- net W: now also R8.1, R8.2, U7.1 (¨RS+), U7.8 (RS)
- net TCC0_CH2/Switch 3 renamed TCC0_CH2/CAN0Switch 3
- new net: C45.1, U17.3 (HB)
- new net CAN1_STANDBY: U1.26 (PB13)
- new net HB4_HO: U17.4 (HO), U18.1 (G1(GHS))
- new net HB4_LO: U17.9 (LO), U18.8 (G2(GLD))
- new net X: C45.2, J11.1 (Pin_1), U17.5 (HS), U18.9 (Vphase)
Other:
- note added: "CONx2 (SPI & UART)"
- note removed: "CONx2 (SPI)"
- moved on the sheet: C10, C19, C22, C23, C24, C33, C36, C38, C39, C9, J3, J4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
